File: self_powered_active_load.kicad_pcb (KiCad board)
At the start: 2 copper layers, 159.9 x 99.8 mm, 80 parts, among them J1 Conn_01x05, J2 Conn_01x03, J3 BANANA_CONN, J4 BANANA_CONN, Q1 2SC4117, Q10 BDW94CFP, Q11 2SC4117, Q12 BDW94CFP, Q13 2SC4117, Q14 BDW94CFP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

Commit message: routing 1st version
Parts:
- moved R15 347.9 mm to (253.5, 80.8)
- moved C7 334.3 mm to (240.8, 71.3), turned to 90 degrees
- moved C3 325.3 mm to (216.7, 105.6), turned to 90 degrees
- moved C6 324.5 mm to (224.5, 88.9), turned to 90 degrees
- moved R25 307.4 mm to (219.7, 88.7), turned to 90 degrees
- moved R26 304.2 mm to (219.7, 83.2), turned to 90 degrees
- moved H2 277.5 mm to (254.0, 140.7)
- moved R14 248.3 mm to (246.2, 79.0)
- moved C5 248.3 mm to (256.1, 70.1)
- moved Q3 248.3 mm to (246.1, 72.9)
- moved Q5 248.3 mm to (256.0, 75.7)
- moved R16 248.3 mm to (251.0, 75.7)
- moved R17 248.3 mm to (251.0, 70.1)
- moved R12 241.5 mm to (247.1, 86.1)
- moved R13 241.5 mm to (244.3, 86.2)
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Routing:
- net Net-(Q13-E): track 0.00 -> 12.4 mm
- net Net-(Q13-C): track 0.00 -> 4.22 mm
Other:
- board size 159.9 x 99.8 mm -> 220 x 99.8 mm
