File: self_powered_active_load.kicad_pcb (KiCad board)
At the start: 2 copper layers, 220 x 99.8 mm, 90 parts, among them J1 Conn_01x05, J2 Conn_01x03, J3 BANANA_CONN, J4 BANANA_CONN, Q1 2SC4117, Q10 BDW94CFP, Q11 2SC4117, Q12 BDW94CFP, Q13 2SC4117, Q14 BDW94CFP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

Commit message: error fixed shunts
Parts:
- R27, R29, R31, R33: value 0R22 -> DNP
Changed lines of the file:
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@@
         (effects (font (size 1 1) (thickness 0.15)))
     )
-    (fp_text value "0R22" (at 15.24 5.62) (layer "F.Fab")
+    (fp_text value "DNP" (at 15.24 5.62) (layer "F.Fab")
         (effects (font (size 1 1) (thickness 0.15)))
     )
@@
         (effects (font (size 1 1) (thickness 0.15)))
     )
-    (fp_text value "0R22" (at 15.24 5.62) (layer "F.Fab")
+    (fp_text value "DNP" (at 15.24 5.62) (layer "F.Fab")
         (effects (font (size 1 1) (thickness 0.15)))
     )
@@
         (effects (font (size 1 1) (thickness 0.15)))
     )
-    (fp_text value "0R22" (at 15.24 5.62) (layer "F.Fab")
+    (fp_text value "DNP" (at 15.24 5.62) (layer "F.Fab")
         (effects (font (size 1 1) (thickness 0.15)))
     )
@@
         (effects (font (size 1 1) (thickness 0.15)))
     )
-    (fp_text value "0R22" (at 15.24 5.62) (layer "F.Fab")
+    (fp_text value "DNP" (at 15.24 5.62) (layer "F.Fab")
         (effects (font (size 1 1) (thickness 0.15)))
     )

Commit message: error removed shunt in PCB
Parts:
- removed R27, R29, R31, R33: DNP, Resistor_THT:R_Axial_DIN0922_L20.0mm_D9.0mm_P30.48mm_Horizontal
Routing:
- net GNDA: track 78.4 -> 59.6 mm
- net Net-(Q11-E): track 66.2 -> 63.7 mm
- net Net-(Q7-E): track 134.4 -> 132.1 mm
- net Net-(Q10-C): track 147.4 -> 145.3 mm
