File: self_powered_active_load.kicad_sch (KiCad schematic)
At the start: 80 parts, among them J1 Conn_01x05, J2 Conn_01x03, J3 BANANA_CONN, J4 BANANA_CONN, Q1 2SC4117, Q2 BDW94CFP, Q3 MMBT5401, Q5 MMBT5401, Q6 MMBT5401, U1 LM10CWM

Commit message: test points added
Parts:
- added TP1, TP10, TP2, TP3, TP4, TP5, TP6, TP7, TP8, TP9: TestPoint, TestPoint:TestPoint_Pad_1.0x1.0mm, symbol Connector:TestPoint
Connections:
- net +1V2: now also TP1.1
- net GNDA: now also TP10.1, TP8.1, TP9.1
- net ctrl: now also TP2.1
- net at Q1.2 (E), Q2.2 (C), R33.1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: now also TP7.1
- net at R35.2, R36.2, R37.2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: now also TP3.1
- net at Q1.2 (E), Q2.2 (C), R27.1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: now also TP4.1
- net at Q1.2 (E), Q2.2 (C), R29.1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: now also TP5.1
- net at Q1.2 (E), Q2.2 (C), R31.1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: now also TP6.1

Commit message: some more documentation
Parts:
- renumbered C5 to C4, C8 to C5, C4 to C6, C6 to C7, C7 to C8, TP9 to TP1, TP3 to TP10, TP10 to TP2, TP8 to TP3, TP1 to TP4, TP2 to TP5, TP4 to TP6, TP5 to TP7, TP6 to TP8, TP7 to TP9
Other:
- company: (none) -> Dr. Frank Kirschbaum, Hohenheimer Straße 71A, 70184 Suttgart
